File: mainboard.brd (EAGLE design)
At the start: 85.7 x 54 mm, 121 parts, among them X1 FH12-24S-0.5SH, X3 87438-02

Commit message: [Rev1] Finished board
Parts:
- added C15, C16: (no value), rcl:C0603
- added C17: (no value), eagle-ltspice:C1206
- added R4: 1k, resistor:R0402
- added R5: 10k, resistor:R0402
- added U$8: BQ21040DBVR, lib:6-SOT-23
- added U$9: ALPS_SSSS810701, lib:ALPS_SSSS810701
- moved U$3 84.1 mm to (77.1, 52.3), turned to 270 degrees
- moved X3 26.9 mm to (31.8, 2.67)
- moved U$2 1.72 mm to (75.8, 35.7)
- moved C9 1.72 mm to (65.7, 37.0)
Connections:
- new net N$54: C15.1, U$3.P$1, U$8.P$6
- new net N$55: R5.1, U$8.P$1
- new net N$56: R4.1, U$8.P$4
- new net V+: C16.1, U$8.P$2, U$9.P$1, X3.1
- net GND: now also C15.2, C16.2, C17.2, R4.2, R5.2, U$3.MECH1, U$3.MECH2, U$3.MECH3, U$3.MECH4, U$3.MECH5, U$3.MECH6, U$3.P$5, U$8.P$5
- net VCC: now also C17.1, U$9.P$3; no longer X3.1
Routing:
- net GND: track 0.00 -> 283.8 mm, vias 0 -> 15
- net KEYROW3: track 0.00 -> 161.2 mm, vias 0 -> 2
- net +3V3: track 0.00 -> 142.3 mm, vias 0 -> 6
- net KEYCOL8: track 0.00 -> 114.5 mm, vias 0 -> 1
- net KEYROW1: track 0.00 -> 106.0 mm, vias 0 -> 3
- net V+: track 0.00 -> 104.6 mm, vias 0 -> 2
- net KEYROW2: track 0.00 -> 103.6 mm, vias 0 -> 3
- net KEYCOL10: track 0.00 -> 95.4 mm, vias 0 -> 1
- net KEYROW0: track 0.00 -> 93.6 mm
- net KEYCOL9: track 0.00 -> 92.7 mm, vias 0 -> 1
- net KEYCOL6: track 0.00 -> 92.3 mm, vias 0 -> 4
- net SD_DAT1: track 0.00 -> 85.6 mm, vias 0 -> 2
- net SD_DAT0: track 0.00 -> 85.6 mm, vias 0 -> 2
- net KEYCOL2: track 0.00 -> 80.4 mm, vias 0 -> 5
- net KEYCOL7: track 0.00 -> 77.8 mm, vias 0 -> 5
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- added copper zone on layer 1, net GND
- added copper zone on layer 16, net GND
Other:
- outline, holes or cut-outs redrawn
